File: gamepad.kicad_pcb (KiCad board)
At the start: 2 copper layers, 30 parts, among them SW1_1 SW_SPST_LED, SW1_2 SW_SPST_LED, SW1_3 SW_SPST_LED, SW1_4 SW_SPST_LED, SW2_1 SW_SPST_LED, SW2_2 SW_SPST_LED, SW2_3 SW_SPST_LED, SW2_4 SW_SPST_LED, SW3_1 SW_SPST_LED, SW3_2 SW_SPST_LED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

Commit message: Modified the pcb-ready for first fab
this is the first try of the pcb fab. It is still to be experted into altium, lets see how that goes :S
Parts:
- added H1: 3mm, Keyboard:3mmHole, F.Cu at (66.0, 45.0)
- added H1: 3mm, Keyboard:3mmHole, F.Cu at (66.0, 136.0)
- added H1: 3mm, Keyboard:3mmHole, F.Cu at (135.0, 136.0)
- added H1: 3mm, Keyboard:3mmHole, F.Cu at (135.0, 45.0)
- moved RC1 2.35 mm to (61.0, 131.0)
Routing:
- net C1: track 117.9 -> 116.4 mm
- added copper zone on B.Cu, net GND
- added copper zone on F.Cu, net GND
Changed lines of the file:
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@@
   (general
     (links 94)
-    (no_connects 27)
-    (area 0 0 0 0)
+    (no_connects 3)
+    (area 50.224999 46.224999 147.770002 143.960002)
     (thickness 1.6)
-    (drawings 1)
-    (tracks 210)
+    (drawings 6)
+    (tracks 211)
     (zones 0)
-    (modules 30)
+    (modules 34)
     (nets 17)
   )
@@
     (mod_text_size 1 1)
     (mod_text_width 0.15)
-    (pad_size 4 4)
-    (pad_drill 4)
+    (pad_size 3.3 3.3)
+    (pad_drill 3.048)
     (pad_to_mask_clearance 0.2)
     (aux_axis_origin 0 0)
@@
     (add_net pwmLED)
   )
+  (module Keyboard:3mmHole (layer F.Cu)
+    (at 66 45)
+    (descr "module 1 pin (ou trou mecanique de percage)")
+    (tags DEV)
+    (fp_text reference H1 (at 0 -3.048) (layer F.SilkS)
+      (effects (font (size 1 1) (thickness 0.15)))
+    )
+    (fp_text value 3mm (at 0 3) (layer F.Fab)
+      (effects (font (size 1 1) (thickness 0.15)))
+    )
+    (fp_circle (center 0 0) (end 2 0.8) (layer F.Fab) (width 0.1))
+    (fp_circle (center 0 0) (end 2.6 0) (layer F.CrtYd) (width 0.05))
+    (fp_circle (center 0 0) (end 0 -2.286) (layer F.SilkS) (width 0.12))
+    (pad "" np_thru_hole circle (at 0 0) (size 3.3 3.3) (drill 3.048) (layers *.Cu *.Mask))
+  )
+  (module Keyboard:3mmHole (layer F.Cu)
+    (at 66 136)
+    (descr "module 1 pin (ou trou mecanique de percage)")
+    (tags DEV)
+    (fp_text reference H1 (at 0 -3.048) (layer F.SilkS)
+      (effects (font (size 1 1) (thickness 0.15)))
+    )
+    (fp_text value 3mm (at 0 3) (layer F.Fab)
+      (effects (font (size 1 1) (thickness 0.15)))
+    )
+    (fp_circle (center 0 0) (end 2 0.8) (layer F.Fab) (width 0.1))
+    (fp_circle (center 0 0) (end 2.6 0) (layer F.CrtYd) (width 0.05))
+    (fp_circle (center 0 0) (end 0 -2.286) (layer F.SilkS) (width 0.12))
+    (pad "" np_thru_hole circle (at 0 0) (size 3.3 3.3) (drill 3.048) (layers *.Cu *.Mask))
+  )
+  (module Keyboard:3mmHole (layer F.Cu)
+    (at 135 136)
+    (descr "module 1 pin (ou trou mecanique de percage)")
+    (tags DEV)
+    (fp_text reference H1 (at 0 -3.048) (layer F.SilkS)
+      (effects (font (size 1 1) (thickness 0.15)))
+    )
+    (fp_text value 3mm (at 0 3) (layer F.Fab)
+      (effects (font (size 1 1) (thickness 0.15)))
+    )
+    (fp_circle (center 0 0) (end 2 0.8) (layer F.Fab) (width 0.1))
+    (fp_circle (center 0 0) (end 2.6 0) (layer F.CrtYd) (width 0.05))
+    (fp_circle (center 0 0) (end 0 -2.286) (layer F.SilkS) (width 0.12))
+    (pad "" np_thru_hole circle (at 0 0) (size 3.3 3.3) (drill 3.048) (layers *.Cu *.Mask))
+  )
   (module CherryMX_PCB_DL (layer F.Cu)
     (at 60 82)
@@
   )
   (module Resistors_THT:R_Axial_DIN0207_L6.3mm_D2.5mm_P7.62mm_Horizontal (layer F.Cu)
-    (at 60.96 133.35)
+    (at 61 131)
     (descr "Resistor, Axial_DIN0207 series, Axial, Horizontal, pin pitch=7.62mm, 0.25W = 1/4W, length*diameter=6.3*2.5mm^2, http://cdn-reichelt.de/documents/datenblatt/B400/1_4W%23YAG.pdf")
     (tags "Resistor Axial_DIN0207 series Axial Horizontal pin pitch 7.62mm 0.25W = 1/4W length 6.3mm diameter 2.5mm")
@@
       (effects (font (size 1 1) (thickness 0.15)) (justify mirror))
     )
-    (fp_text value Conn_01x12 (at -4 0 540) (layer B.Fab)
+    (fp_text value Conn_01x12 (at -4 0 360) (layer B.SilkS)
       (effects (font (size 1 1) (thickness 0.15)) (justify mirror))
     )
@@
     (pad "" smd rect (at 3 9.75 270) (size 3 2.1) (layers B.Cu B.Paste B.Mask))
   )
-  (gr_text "GamePad V0.1\nSwitched Board\nJLEM" (at 142.24 134.62 270) (layer F.Cu)
+  (module Keyboard:3mmHole (layer F.Cu)
+    (at 135 45)
+    (descr "module 1 pin (ou trou mecanique de percage)")
+    (tags DEV)
+    (fp_text reference H1 (at 0 -3.048) (layer F.SilkS)
+      (effects (font (size 1 1) (thickness 0.15)))
+    )
+    (fp_text value 3mm (at 0 3) (layer F.Fab)
+      (effects (font (size 1 1) (thickness 0.15)))
+    )
+    (fp_circle (center 0 0) (end 2 0.8) (layer F.Fab) (width 0.1))
+    (fp_circle (center 0 0) (end 2.6 0) (layer F.CrtYd) (width 0.05))
+    (fp_circle (center 0 0) (end 0 -2.286) (layer F.SilkS) (width 0.12))
+    (pad "" np_thru_hole circle (at 0 0) (size 3.3 3.3) (drill 3.048) (layers *.Cu *.Mask))
+  )
+  (gr_line (start 148 129) (end 148 54) (angle 90) (layer F.SilkS) (width 0.2))
+  (gr_line (start 47 54) (end 47 129) (angle 90) (layer F.SilkS) (width 0.2))
+  (gr_line (start 143 39) (end 53 39) (angle 90) (layer F.SilkS) (width 0.2))
+  (dimension 91 (width 0.3) (layer F.SilkS)
+    (gr_text "91.000 mm" (at 48.65 90.5 270) (layer F.SilkS)
+      (effects (font (size 1.5 1.5) (thickness 0.3)))
+    )
+    (feature1 (pts (xy 66 136) (xy 47.3 136)))
+    (feature2 (pts (xy 66 45) (xy 47.3 45)))
+    (crossbar (pts (xy 50 45) (xy 50 136)))
+    (arrow1a (pts (xy 50 136) (xy 49.413579 134.873496)))
+    (arrow1b (pts (xy 50 136) (xy 50.586421 134.873496)))
+    (arrow2a (pts (xy 50 45) (xy 49.413579 46.126504)))
+    (arrow2b (pts (xy 50 45) (xy 50.586421 46.126504)))
+  )
+  (dimension 69 (width 0.3) (layer F.SilkS)
+    (gr_text "69.000 mm" (at 100.5 40.65) (layer F.SilkS)
+      (effects (font (size 1.5 1.5) (thickness 0.3)))
+    )
+    (feature1 (pts (xy 135 45) (xy 135 39.3)))
+    (feature2 (pts (xy 66 45) (xy 66 39.3)))
+    (crossbar (pts (xy 66 42) (xy 135 42)))
+    (arrow1a (pts (xy 135 42) (xy 133.873496 42.586421)))
+    (arrow1b (pts (xy 135 42) (xy 133.873496 41.413579)))
+    (arrow2a (pts (xy 66 42) (xy 67.126504 42.586421)))
+    (arrow2b (pts (xy 66 42) (xy 67.126504 41.413579)))
+  )
+  (gr_text "GamePad V0.1\nSwitched Board\nJLEM" (at 132 130 360) (layer F.Cu)
     (effects (font (size 1 1) (thickness 0.25)))
   )
@@
   (segment (start 67.874 92.872) (end 67.874 73.872) (width 0.5) (layer F.Cu) (net 2))
   (segment (start 67.874 111.872) (end 67.874 92.872) (width 0.5) (layer F.Cu) (net 2))
-  (segment (start 68.58 133.35) (end 68.58 112.578) (width 0.5) (layer F.Cu) (net 2))
+  (segment (start 68.6 130.9) (end 68.58 112.578) (width 0.5) (layer F.Cu) (net 2))
   (segment (start 68.58 112.578) (end 67.874 111.872) (width 0.5) (layer F.Cu) (net 2))
   (segment (start 103.35 135.89) (end 103.35 133.83) (width 0.5) (layer B.Cu) (net 2))
-  (segment (start 71.12 135.89) (end 68.58 133.35) (width 0.5) (layer B.Cu) (net 2))
-  (segment (start 88.9 135.89) (end 71.12 135.89) (width 0.5) (layer B.Cu) (net 2))
+  (segment (start 73.42 135.89) (end 68.58 131.05) (width 0.5) (layer B.Cu) (net 2))
+  (segment (start 88.9 135.89) (end 73.42 135.89) (width 0.5) (layer B.Cu) (net 2))
   (segment (start 91.44 133.35) (end 88.9 135.89) (width 0.5) (layer B.Cu) (net 2))
   (segment (start 102.87 133.35) (end 91.44 133.35) (width 0.5) (layer B.Cu) (net 2))
@@
   (segment (start 107.95 133.35) (end 107.1 134.2) (width 0.5) (layer B.Cu) (net 5))
   (segment (start 107.1 134.2) (end 107.1 135.89) (width 0.5) (layer B.Cu) (net 5))
+  (segment (start 143.51 125.73) (end 140.27 125.73) (width 0.5) (layer B.Cu) (net 6))
+  (segment (start 144.78 125.73) (end 143.51 125.73) (width 0.5) (layer B.Cu) (net 6))
+  (segment (start 129 137) (end 126 137) (width 0.5) (layer B.Cu) (net 6))
+  (segment (start 140.27 125.73) (end 129 137) (width 0.5) (layer B.Cu) (net 6))
   (segment (start 143.874 66.872) (end 143.874 47.872) (width 0.5) (layer F.Cu) (net 6))
   (segment (start 143.874 85.872) (end 143.874 66.872) (width 0.5) (layer F.Cu) (net 6))
@@
   (segment (start 144.78 105.778) (end 143.874 104.872) (width 0.5) (layer F.Cu) (net 6))
   (segment (start 108.35 135.89) (end 113.03 135.89) (width 0.5) (layer B.Cu) (net 6))
-  (segment (start 143.51 125.73) (end 144.78 125.73) (width 0.5) (layer B.Cu) (net 6))
-  (segment (start 132.08 137.16) (end 143.51 125.73) (width 0.5) (layer B.Cu) (net 6))
-  (segment (start 125.73 137.16) (end 132.08 137.16) (width 0.5) (layer B.Cu) (net 6))
   (segment (start 114.3 137.16) (end 125.73 137.16) (width 0.5) (layer B.Cu) (net 6))
   (segment (start 113.03 135.89) (end 114.3 137.16) (width 0.5) (layer B.Cu) (net 6))
@@
   (segment (start 97.79 142.24) (end 86.36 142.24) (width 0.5) (layer B.Cu) (net 15))
   (segment (start 98.35 141.68) (end 97.79 142.24) (width 0.5) (layer B.Cu) (net 15))
+  (zone (net 1) (net_name GND) (layer B.Cu) (hatch edge 0.508)
+    (connect_pads (clearance 0.508))
+    (min_thickness 0.254)
+    (fill yes (arc_segments 16) (thermal_gap 0.508) (thermal_bridge_width 0.508) (smoothing chamfer) (radius 0.5))
+    (polygon
+      (pts
+        (xy 148 54) (xy 148 129) (xy 143 145) (xy 53 145) (xy 47 129)
+        (xy 47 54) (xy 53 39) (xy 143 39)
+      )
+    )
+  )
+  (zone (net 1) (net_name GND) (layer F.Cu) (hatch edge 0.508)
+    (connect_pads (clearance 0.508))
+    (min_thickness 0.254)
+    (fill yes (arc_segments 16) (thermal_gap 0.508) (thermal_bridge_width 0.508) (smoothing chamfer) (radius 0.5))
+    (polygon
+      (pts
+        (xy 148 54) (xy 148 129) (xy 143 145) (xy 53 145) (xy 47 129)
+        (xy 47 54) (xy 53 39) (xy 143 39)
+      )
+    )
+  )
 )

Commit message: changed some vias
Parts:
- renumbered H1 to H2, H1 to H3, H1 to H4
Routing:
- net pwmLED: track 430.4 -> 451.5 mm, vias 3 -> 2
Other:
- net class Default: via_dia 0.6 -> 0.8
- rule trace_min: 0.25 -> 0.2
- rule via_min_size: 0.4 -> 0.6
Changed lines of the file:
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@@
-(kicad_pcb (version 4) (host pcbnew 4.0.7-e2-6376~58~ubuntu16.04.1)
+(kicad_pcb (version 20170922) (host pcbnew no-vcs-found-ad9916e~61~ubuntu16.04.1)
   (general
-    (links 94)
-    (no_connects 3)
-    (area 50.224999 46.224999 147.770002 143.960002)
     (thickness 1.6)
     (drawings 6)
-    (tracks 211)
+    (tracks 214)
     (zones 0)
     (modules 34)
@@
     (0 F.Cu signal)
     (31 B.Cu signal)
-    (32 B.Adhes user)
-    (33 F.Adhes user)
-    (34 B.Paste user)
-    (35 F.Paste user)
+    (32 B.Adhes user hide)
+    (33 F.Adhes user hide)
+    (34 B.Paste user hide)
+    (35 F.Paste user hide)
     (36 B.SilkS user)
     (37 F.SilkS user)
-    (38 B.Mask user)
-    (39 F.Mask user)
-    (40 Dwgs.User user)
-    (41 Cmts.User user)
-    (42 Eco1.User user)
-    (43 Eco2.User user)
-    (44 Edge.Cuts user)
-    (45 Margin user)
-    (46 B.CrtYd user)
-    (47 F.CrtYd user)
-    (48 B.Fab user)
-    (49 F.Fab user)
+    (38 B.Mask user hide)
+    (39 F.Mask user hide)
+    (40 Dwgs.User user hide)
+    (41 Cmts.User user hide)
+    (42 Eco1.User user hide)
+    (43 Eco2.User user hide)
+    (44 Edge.Cuts user hide)
+    (45 Margin user hide)
+    (46 B.CrtYd user hide)
+    (47 F.CrtYd user hide)
+    (48 B.Fab user hide)
+    (49 F.Fab user hide)
   )
   (setup
@@
     (zone_clearance 0.508)
     (zone_45_only no)
-    (trace_min 0.25)
+    (trace_min 0.2)
     (segment_width 0.2)
     (edge_width 0.15)
-    (via_size 0.6)
+    (via_size 0.8)
     (via_drill 0.4)
-    (via_min_size 0.4)
+    (via_min_size 0.6)
     (via_min_drill 0.3)
+    (user_via 1 0.4)
     (uvia_size 0.3)
     (uvia_drill 0.1)
@@
     (visible_elements FFFFFF7F)
     (pcbplotparams
-      (layerselection 0x00030_80000001)
+      (layerselection 0x00000_7ffffffe)
       (usegerberextensions false)
+      (usegerberattributes true)
+      (usegerberadvancedattributes true)
+      (creategerberjobfile true)
       (excludeedgelayer true)
       (linewidth 0.100000)
@@
       (hpglpenspeed 20)
       (hpglpendiameter 15)
-      (hpglpenoverlay 2)
       (psnegative false)
       (psa4output false)
@@
       (outputformat 1)
       (mirror false)
-      (drillshape 1)
+      (drillshape 0)
       (scaleselection 1)
-      (outputdirectory ""))
+      (outputdirectory try3/))
   )
   (net 0 "")
@@
     (clearance 0.2)
     (trace_width 0.25)
-    (via_dia 0.6)
+    (via_dia 0.8)
     (via_drill 0.4)
     (uvia_dia 0.3)
@@
     (descr "module 1 pin (ou trou mecanique de percage)")
     (tags DEV)
-    (fp_text reference H1 (at 0 -3.048) (layer F.SilkS)
+    (fp_text reference H2 (at 0 -3.048) (layer F.SilkS)
       (effects (font (size 1 1) (thickness 0.15)))
     )
@@
     (descr "module 1 pin (ou trou mecanique de percage)")
     (tags DEV)
-    (fp_text reference H1 (at 0 -3.048) (layer F.SilkS)
+    (fp_text reference H3 (at 0 -3.048) (layer F.SilkS)
       (effects (font (size 1 1) (thickness 0.15)))
     )
@@
     (descr "module 1 pin (ou trou mecanique de percage)")
     (tags DEV)
-    (fp_text reference H1 (at 0 -3.048) (layer F.SilkS)
+    (fp_text reference H4 (at 0 -3.048) (layer F.SilkS)
       (effects (font (size 1 1) (thickness 0.15)))
     )
@@
   (module Keyboard:Molex_Right_Angle_1.25_mm_12_Contacts (layer B.Cu)
     (at 101.6 135.89 270)
-    (fp_text reference uCint1 (at 1.75 1.25 360) (layer B.SilkS)
+    (fp_text reference uCint1 (at 1.75 1.25) (layer B.SilkS)
       (effects (font (size 1 1) (thickness 0.15)) (justify mirror))
     )
-    (fp_text value Conn_01x12 (at -4 0 360) (layer B.SilkS)
+    (fp_text value Conn_01x12 (at -4 0) (layer B.SilkS)
       (effects (font (size 1 1) (thickness 0.15)) (justify mirror))
     )
@@
     (arrow2b (pts (xy 66 42) (xy 67.126504 41.413579)))
   )
-  (gr_text "GamePad V0.1\nSwitched Board\nJLEM" (at 132 130 360) (layer F.Cu)
+  (gr_text "GamePad V0.1\nSwitched Board\nJLEM" (at 132 130) (layer F.Cu)
     (effects (font (size 1 1) (thickness 0.25)))
   )
@@
   (segment (start 58.3 53.46) (end 75.19 53.46) (width 0.5) (layer B.Cu) (net 7))
   (segment (start 56.19 55.57) (end 58.3 53.46) (width 0.5) (layer B.Cu) (net 7))
+  (via (at 96.52 139.7) (size 1) (drill 0.4) (layers F.Cu B.Cu) (net 8))
+  (segment (start 97.1 139.12) (end 96.52 139.7) (width 0.5) (layer B.Cu) (net 8))
+  (segment (start 96.52 139.7) (end 95.25 138.43) (width 0.5) (layer F.Cu) (net 8))
+  (segment (start 95.25 138.43) (end 95.25 119.433) (width 0.5) (layer F.Cu) (net 8))
+  (segment (start 96.603 118.08) (end 95.25 119.433) (width 0.5) (layer F.Cu) (net 8))
+  (segment (start 97.1 139.12) (end 97.1 135.89) (width 0.5) (layer B.Cu) (net 8))
+  (via (at 69.85 125.73) (size 1) (drill 0.4) (layers F.Cu B.Cu) (net 8))
+  (segment (start 69.85 125.73) (end 68.58 127) (width 0.5) (layer B.Cu) (net 8))
+  (segment (start 68.58 127) (end 59.69 127) (width 0.5) (layer B.Cu) (net 8))
+  (segment (start 59.69 127) (end 58.603 125.913) (width 0.5) (layer B.Cu) (net 8))
+  (segment (start 58.603 125.08) (end 58.603 125.913) (width 0.5) (layer B.Cu) (net 8))
+  (segment (start 69.85 125.73) (end 77.5 118.08) (width 0.5) (layer F.Cu) (net 8))
+  (segment (start 96.483 60.96) (end 95.25 60.96) (width 0.5) (layer B.Cu) (net 8) (status 400000))
+  (segment (start 95.25 60.96) (end 92.71 63.5) (width 0.5) (layer B.Cu) (net 8))
+  (segment (start 92.71 63.5) (end 80.023 63.5) (width 0.5) (layer B.Cu) (net 8))
+  (segment (start 80.023 63.5) (end 77.603 61.08) (width 0.5) (layer B.Cu) (net 8))
+  (segment (start 96.483 60.96) (end 96.603 61.08) (width 0.5) (layer B.Cu) (net 8) (status C00000))
+  (segment (start 115.603 99.08) (end 115.603 99.093) (width 0.5) (layer B.Cu) (net 8) (status C00000))
+  (segment (start 115.603 99.093) (end 118.11 101.6) (width 0.5) (layer B.Cu) (net 8) (status 400000))
+  (segment (start 132.083 101.6) (end 134.603 99.08) (width 0.5) (layer B.Cu) (net 8) (status 800000))
+  (segment (start 118.11 101.6) (end 132.083 101.6) (width 0.5) (layer B.Cu) (net 8))
   (segment (start 77.603 118.08) (end 77.5 118.08) (width 0.5) (layer F.Cu) (net 8))
-  (segment (start 77.5 118.08) (end 69.85 125.73) (width 0.5) (layer F.Cu) (net 8))
-  (segment (start 58.603 125.913) (end 58.603 125.08) (width 0.5) (layer B.Cu) (net 8))
-  (segment (start 59.69 127) (end 58.603 125.913) (width 0.5) (layer B.Cu) (net 8))
-  (segment (start 68.58 127) (end 59.69 127) (width 0.5) (layer B.Cu) (net 8))
-  (segment (start 69.85 125.73) (end 68.58 127) (width 0.5) (layer B.Cu) (net 8))
-  (via (at 69.85 125.73) (size 0.6) (drill 0.4) (layers F.Cu B.Cu) (net 8))
   (segment (start 96.603 118.08) (end 96.55 118.08) (width 0.5) (layer B.Cu) (net 8))
   (segment (start 96.55 118.08) (end 93.98 120.65) (width 0.5) (layer B.Cu) (net 8))
@@
   (segment (start 99.06 63.5) (end 113.183 63.5) (width 0.5) (layer B.Cu) (net 8))
   (segment (start 77.603 61.08) (end 77.603 62.097) (width 0.5) (layer B.Cu) (net 8))
+  (segment (start 77.603 62.097) (end 68.58 71.12) (width 0.5) (layer B.Cu) (net 8))
+  (segment (start 68.58 71.12) (end 61.643 71.12) (width 0.5) (layer B.Cu) (net 8))
   (segment (start 61.643 71.12) (end 58.603 68.08) (width 0.5) (layer B.Cu) (net 8))
-  (segment (start 68.58 71.12) (end 61.643 71.12) (width 0.5) (layer B.Cu) (net 8))
-  (segment (start 77.603 62.097) (end 68.58 71.12) (width 0.5) (layer B.Cu) (net 8))
-  (segment (start 96.603 61.08) (end 95.37 61.08) (width 0.5) (layer F.Cu) (net 8))
-  (segment (start 80.023 63.5) (end 77.603 61.08) (width 0.5) (layer B.Cu) (net 8))
-  (segment (start 92.71 63.5) (end 80.023 63.5) (width 0.5) (layer B.Cu) (net 8))
-  (segment (start 95.25 60.96) (end 92.71 63.5) (width 0.5) (layer B.Cu) (net 8))
-  (via (at 95.25 60.96) (size 0.6) (drill 0.4) (layers F.Cu B.Cu) (net 8))
-  (segment (start 95.37 61.08) (end 95.25 60.96) (width 0.5) (layer F.Cu) (net 8))
   (segment (start 96.603 80.08) (end 94.05 80.08) (width 0.5) (layer F.Cu) (net 8))
   (segment (start 91.44 66.243) (end 96.603 61.08) (width 0.5) (layer F.Cu) (net 8))
@@
   (segment (start 91.44 116.84) (end 91.44 104.243) (width 0.5) (layer F.Cu) (net 8))
   (segment (start 92.68 118.08) (end 91.44 116.84) (width 0.5) (layer F.Cu) (net 8))
-  (segment (start 97.1 135.89) (end 97.1 139.12) (width 0.5) (layer B.Cu) (net 8))
-  (segment (start 95.25 119.433) (end 96.603 118.08) (width 0.5) (layer F.Cu) (net 8))
-  (segment (start 95.25 138.43) (end 95.25 119.433) (width 0.5) (layer F.Cu) (net 8))
-  (segment (start 96.52 139.7) (end 95.25 138.43) (width 0.5) (layer F.Cu) (net 8))
-  (via (at 96.52 139.7) (size 0.6) (drill 0.4) (layers F.Cu B.Cu) (net 8))
-  (segment (start 97.1 139.12) (end 96.52 139.7) (width 0.5) (layer B.Cu) (net 8))
   (segment (start 121.92 133.35) (end 120.65 134.62) (width 0.5) (layer B.Cu) (net 9))
   (segment (start 146.05 120.65) (end 146.05 92.71) (width 0.5) (layer B.Cu) (net 9))
